Commit message: car model

File: src/ackermann_vehicle/ackermann_vehicle_description/urdf/em_3905.urdf.xacro (robot description, xacro)
@@ -99,7 +99,4 @@
     <color rgba="0.5 0.5 0.5 1"/>
   </material>
-  <material name="tire_mat">
-    <color rgba="0 0 0 1"/>
-  </material>
   <!-- Null inertial element. This is needed to make the model work with
        Gazebo. -->
@@ -242,7 +239,6 @@
                      0"/>
         <geometry>
-          <cylinder radius="${tire_dia / 2}" length="${tire_width}"/>
-        </geometry>
-        <material name="tire_mat"/>
+          <mesh filename="package://ackermann_vehicle_description/meshes/tire.dae"/>
+        </geometry>
       </visual>
       <collision>
@@ -259,7 +255,4 @@
           height="${tire_width}" mass="${wheel_mass}"/>
     </link>
-    <gazebo reference="${lr_prefix}_${fr_prefix}_wheel">
-      <material>Gazebo/Black</material>
-    </gazebo>
   </xacro:macro>
   <!-- Front wheel -->
@@ -321,7 +314,7 @@
       <origin xyz="0 0 ${-chassis_height / 2}"/>
       <geometry>
-        <box size="${chassis_length} ${chassis_width} ${chassis_height}"/>
+        <!--box size="${chassis_length} ${chassis_width} ${chassis_height}"/-->
+        <mesh filename="package://ackermann_vehicle_description/meshes/chassis.dae"/>
       </geometry>
-      <material name="chassis_mat"/>
     </visual>
     <collision>
@@ -337,7 +330,4 @@
     </xacro:solid_cuboid_inertial>
   </link>
-  <gazebo reference="chassis">
-    <material>Gazebo/Grey</material>
-  </gazebo>
   <joint name="base_link_to_chassis" type="fixed">
     <parent link="base_link"/>

Commit message: good model

File: src/ackermann_vehicle/ackermann_vehicle_description/urdf/em_3905.urdf.xacro (robot description, xacro)
@@ -35,6 +35,6 @@
   <xacro:property name="chassis_length" value="0.258"/>
   <xacro:property name="chassis_width" value="0.168"/>
-  <xacro:property name="chassis_height" value="0.01"/>
-  <xacro:property name="chassis_mass" value="2.788"/>
+  <xacro:property name="chassis_height" value="0.05"/>
+  <xacro:property name="chassis_mass" value="3.5"/>
   <!-- battery_dist is the distance between the inner edges of the
        batteries. battery_comp_depth is the battery compartment depth.
@@ -56,5 +56,5 @@
   <xacro:property name="hub_dia" value="0.09652"/>
   <xacro:property name="tire_dia" value="0.14605"/>
-  <xacro:property name="tire_width" value="0.0889"/>
+  <xacro:property name="tire_width" value="0.06"/>
   <xacro:property name="hex_hub_depth" value="0.01445"/>
   <xacro:property name="wheel_mass" value="0.29"/>
@@ -63,5 +63,5 @@
        from a U joint to the corresponding hex hub. wheel_travel is the
        vertical wheel travel. -->
-  <xacro:property name="wheelbase" value="0.335"/>
+  <xacro:property name="wheelbase" value="0.42"/>
   <xacro:property name="hex_hub_dist" value="0.365"/>
   <xacro:property name="axle_length" value="0.03"/>
@@ -72,5 +72,5 @@
        of a Traxxas Ultra Shock shock absorber spring's constant, is
        437.817 N/m. -->
-  <xacro:property name="shock_eff_limit" value="12.5106"/>
+  <xacro:property name="shock_eff_limit" value="22.5106"/>
   <xacro:property name="shock_vel_limit" value="1000"/>
   <!-- The specifications for a Titan(R) 550 motor could not be found, so the
@@ -93,10 +93,10 @@
   <xacro:property name="servo_stall_torque" value="0.5649"/>
   <xacro:property name="servo_no_load_speed" value="4.553"/>
-  <material name="battery_mat">
+  <!--material name="battery_mat">
     <color rgba="0 0 1 1"/>
   </material>
   <material name="chassis_mat">
     <color rgba="0.5 0.5 0.5 1"/>
-  </material>
+  </material-->
   <!-- Null inertial element. This is needed to make the model work with
        Gazebo. -->

Commit message: tire width fix

File: src/ackermann_vehicle/ackermann_vehicle_description/urdf/em_3905.urdf.xacro (robot description, xacro)
@@ -56,5 +56,5 @@
   <xacro:property name="hub_dia" value="0.09652"/>
   <xacro:property name="tire_dia" value="0.14605"/>
-  <xacro:property name="tire_width" value="0.06"/>
+  <xacro:property name="tire_width" value="0.0855"/>
   <xacro:property name="hex_hub_depth" value="0.01445"/>
   <xacro:property name="wheel_mass" value="0.29"/>

Commit message: good model

File: src/ackermann_vehicle/ackermann_vehicle_description/urdf/em_3905.urdf.xacro (robot description, xacro)
@@ -351,5 +351,5 @@
   <link name="hokuyo_sensor_link" type="laser">
     <visual>
-      <origin xyz="0 0 -0.02" rpy="3.14 3.14 3.14"/>
+      <origin xyz="0 0 0" rpy="3.14 3.14 3.14"/>
       <geometry>
         <mesh filename="package://gazebo_plugins/test/multi_robot_scenario/meshes/laser/hokuyo.dae"/>
@@ -364,5 +364,5 @@
   </link>
   <joint name="laser_to_base" type="fixed">
-    <origin xyz="-0.15 0 0.2"/>
+    <origin xyz="-0.15 0 0.13"/>
     <parent link="base_link" />
     <child link="hokuyo_sensor_link"/>

Commit message: top view camera

File: src/ackermann_vehicle/ackermann_vehicle_description/urdf/em_3905.urdf.xacro (robot description, xacro)
@@ -428,3 +428,71 @@
     </plugin>
   </gazebo>
+  <!-- camera -->
+  <xacro:property name="camera_link" value="0.05" /> <!-- Size of square 'camera' box -->
+  <joint name="camera_joint" type="fixed">
+    <axis xyz="0 1 0" />
+    <origin xyz="-0.5 0 0.5" rpy="0 0.5 0"/>
+    <parent link="base_link"/>
+    <child link="camera_link"/>
+  </joint>
+  <!-- Camera -->
+  <link name="camera_link">
+    <collision>
+      <origin xyz="0 0 0" rpy="0 0 0"/>
+      <geometry>
+    <box size="${camera_link} ${camera_link} ${camera_link}"/>
+      </geometry>
+    </collision>
+    <!--visual>
+      <origin xyz="0 0 0" rpy="0 0 0"/>
+      <geometry>
+    <box size="${camera_link} ${camera_link} ${camera_link}"/>
+      </geometry>
+      <material name="red"/>
+    </visual-->
+    <inertial>
+      <mass value="1e-5" />
+      <origin xyz="0 0 0" rpy="0 0 0"/>
+      <inertia ixx="1e-6" ixy="0" ixz="0" iyy="1e-6" iyz="0" izz="1e-6" />
+    </inertial>
+  </link>
+  <gazebo reference="camera_link">
+    <sensor type="camera" name="top_view">
+      <update_rate>30.0</update_rate>
+      <camera name="head">
+        <horizontal_fov>1.3962634</horizontal_fov>
+        <image>
+          <width>640</width>
+          <height>480</height>
+          <format>R8G8B8</format>
+        </image>
+        <clip>
+          <near>0.02</near>
+          <far>300</far>
+        </clip>
+        <noise>
+          <type>gaussian</type>
+          <!-- Noise is sampled independently per pixel on each frame.
+               That pixel's noise value is added to each of its color
+               channels, which at that point lie in the range [0,1]. -->
+          <mean>0.0</mean>
+          <stddev>0.007</stddev>
+        </noise>
+      </camera>
+      <!--plugin name="camera_controller" filename="libgazebo_ros_camera.so">
+        <alwaysOn>true</alwaysOn>
+        <updateRate>0.0</updateRate>
+        <cameraName>top_cam</cameraName>
+        <imageTopicName>image_raw</imageTopicName>
+        <cameraInfoTopicName>camera_info</cameraInfoTopicName>
+        <frameName>camera_link</frameName>
+        <hackBaseline>0.07</hackBaseline>
+        <distortionK1>0.0</distortionK1>
+        <distortionK2>0.0</distortionK2>
+        <distortionK3>0.0</distortionK3>
+        <distortionT1>0.0</distortionT1>
+        <distortionT2>0.0</distortionT2>
+      </plugin-->
+    </sensor>
+  </gazebo>
 </robot>

Commit message: speed estimaton in dnonav

File: src/ackermann_vehicle/ackermann_vehicle_description/urdf/em_3905.urdf.xacro (robot description, xacro)
@@ -444,5 +444,5 @@
       </geometry>
     </collision>
-    <!--visual>
+    <visual>
       <origin xyz="0 0 0" rpy="0 0 0"/>
       <geometry>
@@ -450,5 +450,5 @@
       </geometry>
       <material name="red"/>
-    </visual-->
+    </visual>
     <inertial>
       <mass value="1e-5" />
@@ -480,5 +480,5 @@
         </noise>
       </camera>
-      <!--plugin name="camera_controller" filename="libgazebo_ros_camera.so">
+      <plugin name="camera_controller" filename="libgazebo_ros_camera.so">
         <alwaysOn>true</alwaysOn>
         <updateRate>0.0</updateRate>
@@ -493,5 +493,5 @@
         <distortionT1>0.0</distortionT1>
         <distortionT2>0.0</distortionT2>
-      </plugin-->
+      </plugin>
     </sensor>
   </gazebo>
